Commit message: Add files via upload

File: src/qube_description/urdf/qube.macro.xacro (robot description, xacro)
@@ -46,5 +46,5 @@
     </joint>
     <joint name="motor_joint" type="revolute">
-      <axis xyz="0 0 1" />
+      <axis xyz="0 0 -1" />
       <limit lower="-3.1415" upper="3.1415" effort="10.0" velocity="1.0"/>
       <parent link="stator_link"/>
